Commit message: all sensors funct

File: giraffe_v2_ws/src/giraffe_v2_description/urdf/giraffe_v2.xacro (robot description, xacro)
@@ -718,5 +718,5 @@
   <child link="motor_left_1"/>
 </joint>
-<joint name="Rev6" type="continuous">
+<joint name="Rev6" type="fixed">
   <origin xyz="-0.03 0.0 -0.0089" rpy="0 0 0"/>
   <parent link="caster_base_1"/>
@@ -724,5 +724,5 @@
   <axis xyz="0.0 -0.0 -1.0"/>
 </joint>
-<joint name="Rev7" type="continuous">
+<joint name="Rev7" type="fixed">
   <origin xyz="-0.0285 -0.0 -0.0525" rpy="0 0 0"/>
   <parent link="caster_swivel_1"/>
@@ -730,5 +730,5 @@
   <axis xyz="0.0 1.0 -0.0"/>
 </joint>
-<joint name="joint_wheel_right" type="continuous">
+<joint name="joint_wheel_right" type="fixed">
   <origin xyz="-0.000106 -0.0222 7.5e-05" rpy="0 0 0"/>
   <parent link="motor_right_1"/>
@@ -736,5 +736,5 @@
   <axis xyz="0.0 -1.0 0.0"/>
 </joint>
-<joint name="joint_wheel_left" type="continuous">
+<joint name="joint_wheel_left" type="fixed">
   <origin xyz="0.0 0.0222 0.0" rpy="0 0 0"/>
   <parent link="motor_left_1"/>
